File: breakingboard/breakingboard.kicad_sch (KiCad schematic)
At the start: 39 parts, among them J1 USB_B_Micro, J2 MFC Connector Plus, J3 MFC Connector Minus, J4 Conn_01x04_Pin, Q1 NPN, SW1 SW_SPDT, U1 AMS1117-3.3, U2 STM32F103C8T6, U3 MCP6L01Rx-xOT, Y1 16MHz

Commit message: pushing to save
Parts:
- SW1: footprint Button_Switch_THT:SW_E-Switch_EG1224_SPDT_Angled -> Button_Switch_SMD:SW_SPDT_PCM12
Changed lines of the file:
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@@
       (effects (font (size 1.27 1.27)))
     )
-    (property "Footprint" "Button_Switch_THT:SW_E-Switch_EG1224_SPDT_Angled" (at 209.55 38.1 0)
+    (property "Footprint" "Button_Switch_SMD:SW_SPDT_PCM12" (at 209.55 38.1 0)
       (effects (font (size 1.27 1.27)) hide)
     )
