File: Colossus/Colossus_rev_A/Colossus_rev_A.kicad_sch (KiCad schematic)
At the start: 26 parts, among them J1 SWD, J2 Right Header, J3 Left Header, U1 STM32H523HEY6TR, U3 LD56100DPU33R, Y1 25MHz

Commit message: pushing to save
Parts:
- C1, C10, C11, C12, C13, C14, C2, C3, C4, C5, C6, C7, C8, C9: footprint (none) -> Capacitor_SMD:C_0201_0603Metric
- D1, D2, FB1: footprint (none) -> LED_SMD:LED_0201_0603Metric
- J1: footprint (none) -> Connector_PinHeader_1.00mm:PinHeader_1x04_P1.00mm_Vertical
- J2, J3: footprint (none) -> Connector_PCBEdge:Samtec_MECF-08-0_-L-DV_2x08_P1.27mm_Polarized_Edge
- L1: footprint (none) -> Inductor_SMD:L_APV_ANR252010
- R1, R2: footprint (none) -> Resistor_SMD:R_01005_0402Metric
- Y1: footprint (none) -> Oscillator:Oscillator_SMD_Abracon_ASCO-4Pin_1.6x1.2mm
Other:
- note added: "TODO: x Temperature Sensing Circuit o Strain Sensing Circuit -- skip this rev x IMU Circuit - MFC Communication Out Circuit - MFC Communication In Circuit - Energy Harvesting Circuit After that -- layout"
- note removed: "TODO: x Temperature Sensing Circuit - Strain Sensing Circuit x IMU Circuit - MFC Communication Out Circuit - MFC Communication In Circuit - Energy Harvesting Circuit After that -- layout"
