File: Colossus/Colossus_rev_A/Energy Harvesting.kicad_sch (KiCad schematic)
At the start: 9 parts, among them J4 Conn_01x02, Q1 NMOS, Q2 NMOS, Q3 PMOS, Q4 PMOS

Commit message: pushing to save
Parts:
- removed C18, C19: C, symbol Device:C
- removed D3, D4: 1N914WT, Diode_SMD:D_SOD-523, symbol Diode:1N914WT
- removed J4: Conn_01x02, symbol Connector_Generic:Conn_01x02
- removed Q1, Q2: NMOS, symbol Simulation_SPICE:NMOS
- removed Q3, Q4: PMOS, symbol Simulation_SPICE:PMOS
Other:
- note removed: "IC"
- note removed: "Rectification"
