File: Colossus/Colossus_rev_A/IMU.kicad_sch (KiCad schematic)
At the start: 6 parts, among them U2 LIS3DH

Commit message: pushing to save
Parts:
- C15, C16: footprint (none) -> Capacitor_SMD:C_0201_0603Metric
- R3, R4, R5: footprint (none) -> Resistor_SMD:R_01005_0402Metric
Connections:
- net +3.3V: no longer C15.1, C16.1, R3.1, R4.1, U2.1 (VDD_IO), U2.14 (VDD)
- new net VBUS: C15.1, C16.1, R3.1, R4.1, U2.1 (VDD_IO), U2.14 (VDD)
Other:
- note added: "I think the IMU will blow up with 5V input probably want to step it down to 3.3"
- moved on the sheet: C15, C16, R3, R4, R5, U2
