File: Colossus/Colossus_rev_A/MFC_COMM_IN.kicad_sch (KiCad schematic)
At the start: 5 parts, among them J8 Conn_01x02, U5 MCP6L01Rx-xOT

Commit message: pushing to save
Parts:
- removed J8: Conn_01x02, symbol Connector_Generic:Conn_01x02
- C23: value C -> 125p; footprint (none) -> Capacitor_SMD:C_0201_0603Metric
- R14: value R_US -> 250M; footprint (none) -> Resistor_SMD:R_01005_0402Metric
- R15: value R_US -> 33k; footprint (none) -> Resistor_SMD:R_01005_0402Metric
Connections:
- net MFCA: now reaches R15.1
