File: Colossus/Colossus_rev_A/Strain Sensing.kicad_sch (KiCad schematic)
At the start: 0 parts

Commit message: pushing to save
Other:
- note added: "HA No"
Changed lines of the file:
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@@
-(kicad_sch (version 20230121) (generator eeschema)
-  (paper "A4")
+(kicad_sch
+	(version 20231120)
+	(generator "eeschema")
+	(generator_version "8.0")
+	(paper "A4")
+	(text "HA No"
+		(exclude_from_sim no)
+		(at 26.67 20.32 0)
+		(effects
+			(font
+				(size 5.08 5.08)
+				(thickness 1.016)
+				(bold yes)
+			)
+		)
+	)
 )
