File: Colossus/Colossus_TI_rev_B/Colossus_TI_rev_B.kicad_sch (KiCad schematic)
At the start: 25 parts, among them J1 SWD, J2 MFC Connection Points, J3 Analog Debugging, J4 Power In, Q3 CSD18541F5, Q4 CSD18541F5, SW2 Reset, U1 XMSM0C1104SDYYR, U2 AD9833xRM, U3 MCP6L01Rx-xOT

Commit message: working on miniaturization
Parts:
- added J3: MFC V+, TestPoint:TestPoint_Pad_2.0x2.0mm, symbol Connector_Generic:Conn_01x01
- added J5: Power In (gnd), TestPoint:TestPoint_Pad_2.0x2.0mm, symbol Connector_Generic:Conn_01x01
- C10: footprint Capacitor_SMD:C_0201_0603Metric -> Capacitor_SMD:C_0805_2012Metric
- J2: value MFC Connection Points -> MFC GND; footprint Connector_PinSocket_2.54mm:PinSocket_1x02_P2.54mm_Vertical -> TestPoint:TestPoint_Pad_2.0x2.0mm; symbol Connector_Generic:Conn_01x02 -> Connector_Generic:Conn_01x01
- J4: value Power In -> Power In (v+); footprint Connector_PinSocket_2.54mm:PinSocket_1x02_P2.54mm_Vertical -> TestPoint:TestPoint_Pad_2.0x2.0mm; symbol Connector_Generic:Conn_01x02 -> Connector_Generic:Conn_01x01
- R7: footprint Resistor_SMD:R_0201_0603Metric -> Resistor_SMD:R_0805_2012Metric
- TH1: footprint Resistor_SMD:R_0805_2012Metric -> Resistor_SMD:R_0402_1005Metric
- renumbered J3 to J6
Connections:
- net GND: now also J5.1 (Pin_1); no longer J4.2 (Pin_2)
- net MFC IN: now also J3.1 (Pin_1); no longer J2.2 (Pin_2)
Changed lines of the file:
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@@
 	)
 	(rectangle
+		(start 160.02 44.45)
+		(end 190.5 59.69)
+		(stroke
+			(width 0)
+			(type default)
+		)
+		(fill
+			(type none)
+		)
+	)
+	(rectangle
 		(start 339.09 105.41)
 		(end 354.33 113.03)
@@
 	)
 	(rectangle
+		(start 160.02 60.96)
+		(end 190.5 81.28)
+		(stroke
+			(width 0)
+			(type default)
+		)
+		(fill
+			(type none)
+		)
+	)
+	(rectangle
 		(start 354.33 135.89)
 		(end 402.59 143.51)
@@
 	(wire
 		(pts
-			(xy 167.64 71.12) (xy 165.1 71.12)
+			(xy 167.64 73.66) (xy 163.83 73.66)
 		)
 		(stroke
@@
 	(wire
 		(pts
-			(xy 163.83 68.58) (xy 163.83 67.31)
-		)
-		(stroke
-			(width 0)
-			(type default)
-		)
-	)
-	(wire
-		(pts
 			(xy 26.67 71.12) (xy 36.83 71.12)
 		)
@@
 	(wire
 		(pts
-			(xy 165.1 71.12) (xy 165.1 72.39)
+			(xy 163.83 73.66) (xy 163.83 74.93)
 		)
 		(stroke
@@
 	(wire
 		(pts
+			(xy 176.53 49.53) (xy 177.8 49.53)
+		)
+		(stroke
+			(width 0)
+			(type default)
+		)
+	)
+	(wire
+		(pts
 			(xy 104.14 226.06) (xy 104.14 231.14)
 		)
@@
 	(global_label "MFC IN"
 		(shape input)
-		(at 176.53 53.34 0)
+		(at 177.8 49.53 0)
 		(fields_autoplaced yes)
 		(effects
@@
 		)
 		(property "Intersheetrefs" "${INTERSHEET_REFS}"
-			(at 186.2281 53.34 0)
+			(at 187.4981 49.53 0)
 			(effects
 				(font
@@
 		(on_board yes)
 		(dnp no)
-		(property "Reference" "J3"
+		(property "Reference" "J6"
 			(at 207.772 57.658 0)
 			(effects
@@
 			(project ""
 				(path "/431f3e11-5eb2-41ca-8e1a-a926513e4d37"
-					(reference "J3")
+					(reference "J6")
 					(unit 1)
 				)
@@
 	)
 	(symbol
-		(lib_id "Connector_Generic:Conn_01x02")
+		(lib_id "Connector_Generic:Conn_01x01")
 		(at 172.72 68.58 0)
 		(unit 1)
@@
 		(fields_autoplaced yes)
 		(property "Reference" "J4"
-			(at 175.26 68.5799 0)
+			(at 175.26 67.3099 0)
 			(effects
 				(font
@@
 			)
 		)
-		(property "Value" "Power In"
-			(at 175.26 71.1199 0)
+		(property "Value" "Power In (v+)"
+			(at 175.26 69.8499 0)
 			(effects
 				(font
@@
 			)
 		)
-		(property "Footprint" "Connector_PinSocket_2.54mm:PinSocket_1x02_P2.54mm_Vertical"
+		(property "Footprint" "TestPoint:TestPoint_Pad_2.0x2.0mm"
 			(at 172.72 68.58 0)
 			(effects
@@
 			)
 		)
-		(property "Description" "Generic connector, single row, 01x02, script generated (kicad-library-utils/schlib/autogen/connector/)"
+		(property "Description" "Generic connector, single row, 01x01, script generated (kicad-library-utils/schlib/autogen/connector/)"
 			(at 172.72 68.58 0)
 			(effects
@@
 		(pin "1"
 		)
-		(pin "2"
-		)
 		(instances
 			(project "Colossus_TI_rev_A"
@@
 	)
 	(symbol
+		(lib_id "Connector_Generic:Conn_01x01")
+		(at 172.72 73.66 0)
+		(unit 1)
+		(exclude_from_sim no)
+		(in_bom yes)
+		(on_board yes)
+		(dnp no)
+		(fields_autoplaced yes)
+		(property "Reference" "J5"
+			(at 175.26 72.3899 0)
+			(effects
+				(font
+					(size 1.27 1.27)
+				)
+				(justify left)
+			)
+		)
+		(property "Value" "Power In (gnd)"
+			(at 175.26 74.9299 0)
+			(effects
+				(font
+					(size 1.27 1.27)
+				)
+				(justify left)
+			)
+		)
+		(property "Footprint" "TestPoint:TestPoint_Pad_2.0x2.0mm"
+			(at 172.72 73.66 0)
+			(effects
+				(font
+					(size 1.27 1.27)
+				)
+				(hide yes)
+			)
+		)
+		(property "Datasheet" "~"
+			(at 172.72 73.66 0)
+			(effects
+				(font
+					(size 1.27 1.27)
+				)
+				(hide yes)
+			)
+		)
+		(property "Description" "Generic connector, single row, 01x01, script generated (kicad-library-utils/schlib/autogen/connector/)"
+			(at 172.72 73.66 0)
+			(effects
+				(font
+					(size 1.27 1.27)
+				)
+				(hide yes)
+			)
+		)
+		(pin "1"
+		)
+		(instances
+			(project "Colossus_TI_rev_B"
+				(path "/431f3e11-5eb2-41ca-8e1a-a926513e4d37"
+					(reference "J5")
+					(unit 1)
+				)
+			)
+		)
+	)
+	(symbol
 		(lib_id "power:GND")
-		(at 165.1 72.39 0)
+		(at 163.83 74.93 0)
 		(unit 1)
 		(exclude_from_sim no)
@@
 		(fields_autoplaced yes)
 		(property "Reference" "#PWR018"
-			(at 165.1 78.74 0)
+			(at 163.83 81.28 0)
 			(effects
 				(font
@@
 		)
 		(property "Value" "GND"
-			(at 165.1 77.47 0)
+			(at 163.83 80.01 0)
 			(effects
 				(font
@@
 		)
 		(property "Footprint" ""
-			(at 165.1 72.39 0)
+			(at 163.83 74.93 0)
 			(effects
 				(font
@@
 		)
 		(property "Datasheet" ""
-			(at 165.1 72.39 0)
+			(at 163.83 74.93 0)
 			(effects
 				(font
@@
 		)
 		(property "Description" "Power symbol creates a global label with name \"GND\" , ground"
-			(at 165.1 72.39 0)
+			(at 163.83 74.93 0)
 			(effects
 				(font
@@
 			)
 		)
-		(property "Footprint" "Capacitor_SMD:C_0201_0603Metric"
+		(property "Footprint" "Capacitor_SMD:C_0805_2012Metric"
 			(at 233.68 115.2652 0)
 			(effects
@@
 	)
 	(symbol
-		(lib_id "Connector_Generic:Conn_01x02")
+		(lib_id "Connector_Generic:Conn_01x01")
 		(at 171.45 55.88 180)
 		(unit 1)
@@
 		(on_board yes)
 		(dnp no)
-		(fields_autoplaced yes)
 		(property "Reference" "J2"
-			(at 171.45 46.99 0)
+			(at 168.148 54.864 0)
 			(effects
 				(font
@@
 			)
 		)
-		(property "Value" "MFC Connection Points"
-			(at 171.45 49.53 0)
+		(property "Value" "MFC GND"
+			(at 165.1 57.404 0)
 			(effects
 				(font
@@
 			)
 		)
-		(property "Footprint" "Connector_PinSocket_2.54mm:PinSocket_1x02_P2.54mm_Vertical"
+		(property "Footprint" "TestPoint:TestPoint_Pad_2.0x2.0mm"
 			(at 171.45 55.88 0)
 			(effects
@@
 			)
 		)
-		(property "Description" "Generic connector, single row, 01x02, script generated (kicad-library-utils/schlib/autogen/connector/)"
+		(property "Description" "Generic connector, single row, 01x01, script generated (kicad-library-utils/schlib/autogen/connector/)"
 			(at 171.45 55.88 0)
 			(effects
@@
 		(pin "1"
 		)
-		(pin "2"
-		)
 		(instances
 			(project ""
@@
 	(symbol
 		(lib_id "power:GND")
-		(at 179.07 55.88 0)
+		(at 179.07 55.88 90)
 		(unit 1)
 		(exclude_from_sim no)
@@
 		(fields_autoplaced yes)
 		(property "Reference" "#PWR16"
-			(at 179.07 62.23 0)
+			(at 185.42 55.88 0)
 			(effects
 				(font
@@
 		)
 		(property "Value" "GND"
-			(at 179.07 60.96 0)
+			(at 182.88 55.8799 90)
 			(effects
 				(font
 					(size 1.27 1.27)
 				)
+				(justify right)
 			)
 		)
@@
 	)
 	(symbol
+		(lib_id "Connector_Generic:Conn_01x01")
+		(at 171.45 49.53 180)
+		(unit 1)
+		(exclude_from_sim no)
+		(in_bom yes)
+		(on_board yes)
+		(dnp no)
+		(property "Reference" "J3"
+			(at 168.148 47.244 0)
+			(effects
+				(font
+					(size 1.27 1.27)
+				)
+			)
+		)
+		(property "Value" "MFC V+"
+			(at 165.862 50.038 0)
+			(effects
+				(font
+					(size 1.27 1.27)
+				)
+			)
+		)
+		(property "Footprint" "TestPoint:TestPoint_Pad_2.0x2.0mm"
+			(at 171.45 49.53 0)
+			(effects
+				(font
+					(size 1.27 1.27)
+				)
+				(hide yes)
+			)
+		)
+		(property "Datasheet" "~"
+			(at 171.45 49.53 0)
+			(effects
+				(font
+					(size 1.27 1.27)
+				)
+				(hide yes)
+			)
+		)
+		(property "Description" "Generic connector, single row, 01x01, script generated (kicad-library-utils/schlib/autogen/connector/)"
+			(at 171.45 49.53 0)
+			(effects
+				(font
+					(size 1.27 1.27)
+				)
+				(hide yes)
+			)
+		)
+		(pin "1"
+		)
+		(instances
+			(project "Colossus_TI_rev_B"
+				(path "/431f3e11-5eb2-41ca-8e1a-a926513e4d37"
+					(reference "J3")
+					(unit 1)
+				)
+			)
+		)
+	)
+	(symbol
 		(lib_id "power:GND")
 		(at 242.57 114.3 0)
@@
 			)
 		)
-		(property "Footprint" "Resistor_SMD:R_0805_2012Metric"
+		(property "Footprint" "Resistor_SMD:R_0402_1005Metric"
 			(at 185.42 166.37 0)
 			(effects
@@
 			)
 		)
-		(property "Footprint" "Resistor_SMD:R_0201_0603Metric"
+		(property "Footprint" "Resistor_SMD:R_0805_2012Metric"
 			(at 212.344 113.284 90)
 			(effects
@@
 	(symbol
 		(lib_id "power:+3.3V")
-		(at 163.83 67.31 0)
+		(at 163.83 68.58 0)
 		(unit 1)
 		(exclude_from_sim no)
@@
 		(fields_autoplaced yes)
 		(property "Reference" "#PWR017"
-			(at 163.83 71.12 0)
+			(at 163.83 72.39 0)
 			(effects
 				(font
@@
 		)
 		(property "Value" "+3.3V"
-			(at 163.83 62.23 0)
+			(at 163.83 63.5 0)
 			(effects
 				(font
@@
 		)
 		(property "Footprint" ""
-			(at 163.83 67.31 0)
+			(at 163.83 68.58 0)
 			(effects
 				(font
@@
 		)
 		(property "Datasheet" ""
-			(at 163.83 67.31 0)
+			(at 163.83 68.58 0)
 			(effects
 				(font
@@
 		)
 		(property "Description" "Power symbol creates a global label with name \"+3.3V\""
-			(at 163.83 67.31 0)
+			(at 163.83 68.58 0)
 			(effects
 				(font

Commit message: final and manufactured draft of revB board
Parts:
- removed Q3, Q4: CSD18541F5, CSD18541F5 - n channel mosfet:DFN149X73X35-3N, symbol CSD18541F5:CSD18541F5
- added H1, H2: MountingHole, MountingHole:MountingHole_2.2mm_M2_Pad_Via, symbol Mechanical:MountingHole
- added U4: SN74LVC1G3157DSFR, Analog Switch - SN74LVC1G3157DSFR:SON35P100X100X40-6N, symbol SN74LVC1G3157DSFR:SN74LVC1G3157DSFR
- C1, C6, C8: footprint Capacitor_SMD:C_0201_0603Metric -> Capacitor_SMD:C_0402_1005Metric
- R4: footprint Resistor_SMD:R_0201_0603Metric -> Resistor_SMD:R_0402_1005Metric
- SW2: footprint button:SW_B3F-1000_OMR -> footprints:SW_B3F-1000_OMR
- U1: footprint footprints:SOT-23-THIN16_DYY_TEX-M -> MSMP0:SOT-23-THIN16_DYY_TEX
Connections:
- net FMout is gone; now on net Charge Amp In: U2.10 (VOUT)
- net MFC IN is gone; now on net Charge Amp In: J3.1 (Pin_1)
- net +3.3V: now also U4.4 (A), U4.5 (VCC); no longer C4.2, C5.2, C6.2, C7.1, U2.2 (VDD), U2.3 (CAP/2.5V), U3.2 (V+)
- net GND: now also U4.2 (GND)
- net PA2 renamed Mode Select
- net Mode Select: now also U4.6 (S)
- new net FM Power: C4.2, C5.2, C6.2, C7.1, U2.2 (VDD), U2.3 (CAP/2.5V), U4.1 (B2)
- new net Strain Power: U3.2 (V+), U4.3 (B1)
Other:
- note added: "Reset"
- note added: "SET( [(R2) / (R1 + R2)]*Vcc1 > vih) of select pin Basically we don't want signals to happen super fast so we slow them down with the pullup pull down RC circut"
- note added: "Switching Modes"
- note added: "analog switch, tri-state buffer, or bidirectional bus switch"
- note removed: "Bidirectional Mosfet Switch to switch between FMout and Strain in THIS IS NOT CORRECT AND NEEDS TO BE FIXED"
- note removed: "Switching Modes and Reset"
- moved on the sheet: C10, R7, SW2
